Commit message: chore: made the robot slightly larger

File: warehouse_sim/urdf/warehouse_robot.urdf.xacro (robot description, xacro)
@@ -4,17 +4,17 @@
   <xacro:arg name="controller_config_path" default=""/>
   <!-- Chassis -->
-  <xacro:property name="base_length" value="0.4"/>
-  <xacro:property name="base_width" value="0.4"/>
-  <xacro:property name="base_height" value="0.12"/>
-  <xacro:property name="base_mass" value="8.0"/>
+  <xacro:property name="base_length" value="0.75"/>
+  <xacro:property name="base_width" value="0.75"/>
+  <xacro:property name="base_height" value="0.25"/>
+  <xacro:property name="base_mass" value="16.0"/>
   <!-- Drive wheels -->
-  <xacro:property name="wheel_radius" value="0.05"/>
-  <xacro:property name="wheel_width" value="0.03"/>
-  <xacro:property name="wheel_mass" value="0.5"/>
+  <xacro:property name="wheel_radius" value="0.1"/>
+  <xacro:property name="wheel_width" value="0.06"/>
+  <xacro:property name="wheel_mass" value="0.75"/>
   <!-- Caster wheels -->
-  <xacro:property name="caster_radius" value="0.025"/>
-  <xacro:property name="caster_mass" value="0.1"/>
+  <xacro:property name="caster_radius" value="0.05"/>
+  <xacro:property name="caster_mass" value="0.2"/>
   <!-- Derived placement offsets -->
-  <xacro:property name="ground_clearance" value="0.02"/>
+  <xacro:property name="ground_clearance" value="0.04"/>
   <xacro:property name="base_z" value="${wheel_radius + ground_clearance}"/>
   <xacro:property name="wheel_z_offset" value="${wheel_radius - base_z}"/>

Commit message: feat: robot box cage and flap

File: warehouse_sim/urdf/warehouse_robot.urdf.xacro (robot description, xacro)
@@ -15,4 +15,10 @@
   <xacro:property name="caster_radius" value="0.05"/>
   <xacro:property name="caster_mass" value="0.2"/>
+  <!-- Cargo cage: thin walls around the chassis, front wall has a hinged flap -->
+  <xacro:property name="cage_wall_height" value="1.0"/>
+  <xacro:property name="cage_wall_thickness" value="0.02"/>
+  <xacro:property name="cage_flap_height" value="0.5"/>
+  <xacro:property name="cage_wall_mass" value="0.5"/>
+  <xacro:property name="cage_flap_mass" value="0.3"/>
   <!-- Derived placement offsets -->
   <xacro:property name="ground_clearance" value="0.04"/>
@@ -21,4 +27,6 @@
   <xacro:property name="caster_z_offset" value="${caster_radius - base_z}"/>
   <xacro:property name="caster_x_offset" value="${base_length / 2 - caster_radius - 0.02}"/>
+  <xacro:property name="cage_base_z" value="${base_height / 2.0}"/>
+  <xacro:property name="cage_front_upper_height" value="${cage_wall_height - cage_flap_height}"/>
   <material name="body_gray">
     <color rgba="0.3 0.3 0.3 1.0"/>
@@ -29,4 +37,7 @@
   <material name="caster_silver">
     <color rgba="0.7 0.7 0.7 1.0"/>
+  </material>
+  <material name="cage_yellow">
+    <color rgba="0.9 0.7 0.1 1.0"/>
   </material>
   <!-- base_footprint sits on the ground and is the robot's control/odometry origin -->
@@ -128,5 +139,89 @@
   <xacro:caster_wheel prefix="front" x_offset="${caster_x_offset}"/>
   <xacro:caster_wheel prefix="back" x_offset="${-caster_x_offset}"/>
-  <!-- ros2_control: only the two driven wheels are actuated -->
+  <!-- Fixed cage wall: a thin box sitting on top of the chassis -->
+  <xacro:macro name="cage_wall" params="name size_x size_y size_z origin_x origin_y origin_z">
+    <link name="${name}_wall_link">
+      <visual>
+        <geometry>
+          <box size="${size_x} ${size_y} ${size_z}"/>
+        </geometry>
+        <material name="cage_yellow"/>
+      </visual>
+      <collision>
+        <geometry>
+          <box size="${size_x} ${size_y} ${size_z}"/>
+        </geometry>
+      </collision>
+      <inertial>
+        <mass value="${cage_wall_mass}"/>
+        <inertia
+          ixx="${cage_wall_mass / 12.0 * (size_y*size_y + size_z*size_z)}" ixy="0" ixz="0"
+          iyy="${cage_wall_mass / 12.0 * (size_x*size_x + size_z*size_z)}" iyz="0"
+          izz="${cage_wall_mass / 12.0 * (size_x*size_x + size_y*size_y)}"/>
+      </inertial>
+    </link>
+    <joint name="${name}_wall_joint" type="fixed">
+      <parent link="base_link"/>
+      <child link="${name}_wall_link"/>
+      <origin xyz="${origin_x} ${origin_y} ${origin_z}" rpy="0 0 0"/>
+    </joint>
+    <gazebo reference="${name}_wall_link">
+      <material>Gazebo/Yellow</material>
+    </gazebo>
+  </xacro:macro>
+  <xacro:cage_wall name="back"
+    size_x="${cage_wall_thickness}" size_y="${base_width}" size_z="${cage_wall_height}"
+    origin_x="${-(base_length/2 - cage_wall_thickness/2)}" origin_y="0"
+    origin_z="${cage_base_z + cage_wall_height/2}"/>
+  <xacro:cage_wall name="left"
+    size_x="${base_length}" size_y="${cage_wall_thickness}" size_z="${cage_wall_height}"
+    origin_x="0" origin_y="${base_width/2 - cage_wall_thickness/2}"
+    origin_z="${cage_base_z + cage_wall_height/2}"/>
+  <xacro:cage_wall name="right"
+    size_x="${base_length}" size_y="${cage_wall_thickness}" size_z="${cage_wall_height}"
+    origin_x="0" origin_y="${-(base_width/2 - cage_wall_thickness/2)}"
+    origin_z="${cage_base_z + cage_wall_height/2}"/>
+  <!-- Front wall: fixed upper section plus a hinged flap covering the bottom cage_flap_height -->
+  <xacro:cage_wall name="front_upper"
+    size_x="${cage_wall_thickness}" size_y="${base_width}" size_z="${cage_front_upper_height}"
+    origin_x="${base_length/2 - cage_wall_thickness/2}" origin_y="0"
+    origin_z="${cage_base_z + cage_flap_height + cage_front_upper_height/2}"/>
+  <!-- Front flap: hinged at its bottom edge, folds down/outward to open like a tailgate -->
+  <link name="front_flap_link">
+    <visual>
+      <origin xyz="0 0 ${cage_flap_height/2}" rpy="0 0 0"/>
+      <geometry>
+        <box size="${cage_wall_thickness} ${base_width} ${cage_flap_height}"/>
+      </geometry>
+      <material name="wheel_black"/>
+    </visual>
+    <collision>
+      <origin xyz="0 0 ${cage_flap_height/2}" rpy="0 0 0"/>
+      <geometry>
+        <box size="${cage_wall_thickness} ${base_width} ${cage_flap_height}"/>
+      </geometry>
+    </collision>
+    <inertial>
+      <origin xyz="0 0 ${cage_flap_height/2}" rpy="0 0 0"/>
+      <mass value="${cage_flap_mass}"/>
+      <inertia
+        ixx="${cage_flap_mass / 12.0 * (base_width*base_width + cage_flap_height*cage_flap_height)}" ixy="0" ixz="0"
+        iyy="${cage_flap_mass / 12.0 * (cage_wall_thickness*cage_wall_thickness + cage_flap_height*cage_flap_height)}" iyz="0"
+        izz="${cage_flap_mass / 12.0 * (cage_wall_thickness*cage_wall_thickness + base_width*base_width)}"/>
+    </inertial>
+  </link>
+  <joint name="front_flap_joint" type="revolute">
+    <parent link="base_link"/>
+    <child link="front_flap_link"/>
+    <origin xyz="${base_length/2 - cage_wall_thickness/2} 0 ${cage_base_z}" rpy="0 0 0"/>
+    <axis xyz="0 1 0"/>
+    <!-- 0 = closed (vertical), pi/2 = fully open (folded flat outward) -->
+    <limit lower="0" upper="${pi/2}" effort="10.0" velocity="1.0"/>
+    <dynamics damping="0.2" friction="0.05"/>
+  </joint>
+  <gazebo reference="front_flap_link">
+    <material>Gazebo/Black</material>
+  </gazebo>
+  <!-- ros2_control: the two driven wheels plus the front cage flap are actuated -->
   <ros2_control name="warehouse_robot_system" type="system">
     <hardware>
@@ -143,4 +238,9 @@
       <state_interface name="velocity"/>
     </joint>
+    <joint name="front_flap_joint">
+      <command_interface name="position"/>
+      <state_interface name="position"/>
+      <state_interface name="velocity"/>
+    </joint>
   </ros2_control>
   <gazebo>

Commit message: feat: camera sensor on robot for april tag vision

File: warehouse_sim/urdf/warehouse_robot.urdf.xacro (robot description, xacro)
@@ -21,4 +21,7 @@
   <xacro:property name="cage_wall_mass" value="0.5"/>
   <xacro:property name="cage_flap_mass" value="0.3"/>
+  <!-- Front RGB camera -->
+  <xacro:property name="camera_size" value="0.04"/>
+  <xacro:property name="camera_mass" value="0.05"/>
   <!-- Derived placement offsets -->
   <xacro:property name="ground_clearance" value="0.04"/>
@@ -223,4 +226,59 @@
     <material>Gazebo/Black</material>
   </gazebo>
+  <!-- Front camera: mounted flush on the chassis front face, below the cage, pointing straight out along +x -->
+  <link name="camera_link">
+    <visual>
+      <geometry>
+        <box size="${camera_size} ${camera_size} ${camera_size}"/>
+      </geometry>
+      <material name="wheel_black"/>
+    </visual>
+    <collision>
+      <geometry>
+        <box size="${camera_size} ${camera_size} ${camera_size}"/>
+      </geometry>
+    </collision>
+    <inertial>
+      <mass value="${camera_mass}"/>
+      <inertia
+        ixx="${camera_mass / 6.0 * camera_size*camera_size}" ixy="0" ixz="0"
+        iyy="${camera_mass / 6.0 * camera_size*camera_size}" iyz="0"
+        izz="${camera_mass / 6.0 * camera_size*camera_size}"/>
+    </inertial>
+  </link>
+  <joint name="camera_joint" type="fixed">
+    <parent link="base_link"/>
+    <child link="camera_link"/>
+    <origin xyz="${base_length/2 + camera_size/2} 0 0" rpy="0 0 0"/>
+  </joint>
+  <!-- Optical frame: REP 103 convention (Z forward, X right, Y down), used for image/camera_info -->
+  <link name="camera_optical_frame"/>
+  <joint name="camera_optical_joint" type="fixed">
+    <parent link="camera_link"/>
+    <child link="camera_optical_frame"/>
+    <origin xyz="0 0 0" rpy="${-pi/2} 0 ${-pi/2}"/>
+  </joint>
+  <gazebo reference="camera_link">
+    <material>Gazebo/Black</material>
+    <sensor name="front_camera" type="camera">
+      <camera>
+        <horizontal_fov>1.4</horizontal_fov>
+        <image>
+          <width>640</width>
+          <height>480</height>
+        </image>
+        <clip>
+          <near>0.05</near>
+          <far>50</far>
+        </clip>
+        <!-- Sensor is aimed straight ahead for now; revisit if the mount angle changes -->
+        <optical_frame_id>camera_optical_frame</optical_frame_id>
+      </camera>
+      <always_on>true</always_on>
+      <update_rate>15</update_rate>
+      <visualize>true</visualize>
+      <topic>front_camera</topic>
+    </sensor>
+  </gazebo>
   <!-- ros2_control: the two driven wheels plus the front cage flap are actuated -->
   <ros2_control name="warehouse_robot_system" type="system">

Commit message: feat: april tag models

File: warehouse_sim/urdf/warehouse_robot.urdf.xacro (robot description, xacro)
@@ -281,4 +281,59 @@
     </sensor>
   </gazebo>
+  <!-- Rear camera: mounted flush on the chassis back face, pointing straight out along -x -->
+  <link name="rear_camera_link">
+    <visual>
+      <geometry>
+        <box size="${camera_size} ${camera_size} ${camera_size}"/>
+      </geometry>
+      <material name="wheel_black"/>
+    </visual>
+    <collision>
+      <geometry>
+        <box size="${camera_size} ${camera_size} ${camera_size}"/>
+      </geometry>
+    </collision>
+    <inertial>
+      <mass value="${camera_mass}"/>
+      <inertia
+        ixx="${camera_mass / 6.0 * camera_size*camera_size}" ixy="0" ixz="0"
+        iyy="${camera_mass / 6.0 * camera_size*camera_size}" iyz="0"
+        izz="${camera_mass / 6.0 * camera_size*camera_size}"/>
+    </inertial>
+  </link>
+  <joint name="rear_camera_joint" type="fixed">
+    <parent link="base_link"/>
+    <child link="rear_camera_link"/>
+    <origin xyz="${-(base_length/2 + camera_size/2)} 0 0" rpy="0 0 ${pi}"/>
+  </joint>
+  <!-- Optical frame: REP 103 convention (Z forward, X right, Y down), used for image/camera_info -->
+  <link name="rear_camera_optical_frame"/>
+  <joint name="rear_camera_optical_joint" type="fixed">
+    <parent link="rear_camera_link"/>
+    <child link="rear_camera_optical_frame"/>
+    <origin xyz="0 0 0" rpy="${-pi/2} 0 ${-pi/2}"/>
+  </joint>
+  <gazebo reference="rear_camera_link">
+    <material>Gazebo/Black</material>
+    <sensor name="rear_camera" type="camera">
+      <camera>
+        <horizontal_fov>1.4</horizontal_fov>
+        <image>
+          <width>640</width>
+          <height>480</height>
+        </image>
+        <clip>
+          <near>0.05</near>
+          <far>50</far>
+        </clip>
+        <!-- Sensor is aimed straight out the back for now; revisit if the mount angle changes -->
+        <optical_frame_id>rear_camera_optical_frame</optical_frame_id>
+      </camera>
+      <always_on>true</always_on>
+      <update_rate>15</update_rate>
+      <visualize>true</visualize>
+      <topic>rear_camera</topic>
+    </sensor>
+  </gazebo>
   <!-- ros2_control: the two driven wheels plus the front cage flap are actuated -->
   <ros2_control name="warehouse_robot_system" type="system">

Commit message: fix: renamed all front camera properties to reflect camera name

File: warehouse_sim/urdf/warehouse_robot.urdf.xacro (robot description, xacro)
@@ -227,5 +227,5 @@
   </gazebo>
   <!-- Front camera: mounted flush on the chassis front face, below the cage, pointing straight out along +x -->
-  <link name="camera_link">
+  <link name="front_camera_link">
     <visual>
       <geometry>
@@ -247,17 +247,17 @@
     </inertial>
   </link>
-  <joint name="camera_joint" type="fixed">
+  <joint name="front_camera_joint" type="fixed">
     <parent link="base_link"/>
-    <child link="camera_link"/>
+    <child link="front_camera_link"/>
     <origin xyz="${base_length/2 + camera_size/2} 0 0" rpy="0 0 0"/>
   </joint>
   <!-- Optical frame: REP 103 convention (Z forward, X right, Y down), used for image/camera_info -->
-  <link name="camera_optical_frame"/>
-  <joint name="camera_optical_joint" type="fixed">
-    <parent link="camera_link"/>
-    <child link="camera_optical_frame"/>
+  <link name="front_camera_optical_frame"/>
+  <joint name="front_camera_optical_joint" type="fixed">
+    <parent link="front_camera_link"/>
+    <child link="front_camera_optical_frame"/>
     <origin xyz="0 0 0" rpy="${-pi/2} 0 ${-pi/2}"/>
   </joint>
-  <gazebo reference="camera_link">
+  <gazebo reference="front_camera_link">
     <material>Gazebo/Black</material>
     <sensor name="front_camera" type="camera">
@@ -273,5 +273,5 @@
         </clip>
         <!-- Sensor is aimed straight ahead for now; revisit if the mount angle changes -->
-        <optical_frame_id>camera_optical_frame</optical_frame_id>
+        <optical_frame_id>front_camera_optical_frame</optical_frame_id>
       </camera>
       <always_on>true</always_on>

Commit message: feat: added imu sensor

File: warehouse_sim/urdf/warehouse_robot.urdf.xacro (robot description, xacro)
@@ -24,4 +24,7 @@
   <xacro:property name="camera_size" value="0.04"/>
   <xacro:property name="camera_mass" value="0.05"/>
+  <!-- IMU -->
+  <xacro:property name="imu_size" value="0.02"/>
+  <xacro:property name="imu_mass" value="0.01"/>
   <!-- Derived placement offsets -->
   <xacro:property name="ground_clearance" value="0.04"/>
@@ -336,4 +339,37 @@
     </sensor>
   </gazebo>
+  <!-- IMU: mounted at the chassis origin -->
+  <link name="imu_link">
+    <visual>
+      <geometry>
+        <box size="${imu_size} ${imu_size} ${imu_size}"/>
+      </geometry>
+      <material name="wheel_black"/>
+    </visual>
+    <collision>
+      <geometry>
+        <box size="${imu_size} ${imu_size} ${imu_size}"/>
+      </geometry>
+    </collision>
+    <inertial>
+      <mass value="${imu_mass}"/>
+      <inertia
+        ixx="${imu_mass / 6.0 * imu_size*imu_size}" ixy="0" ixz="0"
+        iyy="${imu_mass / 6.0 * imu_size*imu_size}" iyz="0"
+        izz="${imu_mass / 6.0 * imu_size*imu_size}"/>
+    </inertial>
+  </link>
+  <joint name="imu_joint" type="fixed">
+    <parent link="base_link"/>
+    <child link="imu_link"/>
+    <origin xyz="0 0 0" rpy="0 0 0"/>
+  </joint>
+  <gazebo reference="imu_link">
+    <sensor name="imu_sensor" type="imu">
+      <always_on>true</always_on>
+      <update_rate>100</update_rate>
+      <topic>imu</topic>
+    </sensor>
+  </gazebo>
   <!-- ros2_control: the two driven wheels plus the front cage flap are actuated -->
   <ros2_control name="warehouse_robot_system" type="system">

Commit message: feat: deleted front camera, replaced with lidar sensor

File: warehouse_sim/urdf/warehouse_robot.urdf.xacro (robot description, xacro)
@@ -21,7 +21,11 @@
   <xacro:property name="cage_wall_mass" value="0.5"/>
   <xacro:property name="cage_flap_mass" value="0.3"/>
-  <!-- Front RGB camera -->
+  <!-- Rear RGB camera -->
   <xacro:property name="camera_size" value="0.04"/>
   <xacro:property name="camera_mass" value="0.05"/>
+  <!-- Front 2D lidar -->
+  <xacro:property name="lidar_radius" value="0.05"/>
+  <xacro:property name="lidar_height" value="0.06"/>
+  <xacro:property name="lidar_mass" value="0.15"/>
   <!-- IMU -->
   <xacro:property name="imu_size" value="0.02"/>
@@ -229,9 +233,10 @@
     <material>Gazebo/Black</material>
   </gazebo>
-  <!-- Front camera: mounted flush on the chassis front face, below the cage, pointing straight out along +x -->
-  <link name="front_camera_link">
+  <!-- Front lidar: centered on the chassis front face, below the cage, so half the puck
+       sticks out past the front edge -->
+  <link name="front_lidar_link">
     <visual>
       <geometry>
-        <box size="${camera_size} ${camera_size} ${camera_size}"/>
+        <cylinder radius="${lidar_radius}" length="${lidar_height}"/>
       </geometry>
       <material name="wheel_black"/>
@@ -239,47 +244,42 @@
     <collision>
       <geometry>
-        <box size="${camera_size} ${camera_size} ${camera_size}"/>
+        <cylinder radius="${lidar_radius}" length="${lidar_height}"/>
       </geometry>
     </collision>
     <inertial>
-      <mass value="${camera_mass}"/>
+      <mass value="${lidar_mass}"/>
       <inertia
-        ixx="${camera_mass / 6.0 * camera_size*camera_size}" ixy="0" ixz="0"
-        iyy="${camera_mass / 6.0 * camera_size*camera_size}" iyz="0"
-        izz="${camera_mass / 6.0 * camera_size*camera_size}"/>
+        ixx="${lidar_mass / 12.0 * (3*lidar_radius*lidar_radius + lidar_height*lidar_height)}" ixy="0" ixz="0"
+        iyy="${lidar_mass / 12.0 * (3*lidar_radius*lidar_radius + lidar_height*lidar_height)}" iyz="0"
+        izz="${lidar_mass / 2.0 * lidar_radius*lidar_radius}"/>
     </inertial>
   </link>
-  <joint name="front_camera_joint" type="fixed">
+  <joint name="front_lidar_joint" type="fixed">
     <parent link="base_link"/>
-    <child link="front_camera_link"/>
-    <origin xyz="${base_length/2 + camera_size/2} 0 0" rpy="0 0 0"/>
-  </joint>
-  <!-- Optical frame: REP 103 convention (Z forward, X right, Y down), used for image/camera_info -->
-  <link name="front_camera_optical_frame"/>
-  <joint name="front_camera_optical_joint" type="fixed">
-    <parent link="front_camera_link"/>
-    <child link="front_camera_optical_frame"/>
-    <origin xyz="0 0 0" rpy="${-pi/2} 0 ${-pi/2}"/>
-  </joint>
-  <gazebo reference="front_camera_link">
+    <child link="front_lidar_link"/>
+    <origin xyz="${base_length/2} 0 0" rpy="0 0 0"/>
+  </joint>
+  <gazebo reference="front_lidar_link">
     <material>Gazebo/Black</material>
-    <sensor name="front_camera" type="camera">
-      <camera>
-        <horizontal_fov>1.4</horizontal_fov>
-        <image>
-          <width>640</width>
-          <height>480</height>
-        </image>
-        <clip>
-          <near>0.05</near>
-          <far>50</far>
-        </clip>
-        <!-- Sensor is aimed straight ahead for now; revisit if the mount angle changes -->
-        <optical_frame_id>front_camera_optical_frame</optical_frame_id>
-      </camera>
+    <sensor name="front_lidar" type="gpu_lidar">
+      <lidar>
+        <scan>
+          <horizontal>
+            <samples>640</samples>
+            <resolution>1</resolution>
+            <min_angle>${-2.0/3.0*pi}</min_angle>
+            <max_angle>${2.0/3.0*pi}</max_angle>
+          </horizontal>
+        </scan>
+        <range>
+          <min>0.1</min>
+          <max>25.0</max>
+          <resolution>0.01</resolution>
+        </range>
+      </lidar>
       <always_on>true</always_on>
-      <update_rate>15</update_rate>
+      <update_rate>10</update_rate>
       <visualize>true</visualize>
-      <topic>front_camera</topic>
+      <topic>front_lidar</topic>
     </sensor>
   </gazebo>

Commit message: chore: made the shelves slightly thinner, robot slightly smaller for increased mobility.

File: warehouse_sim/urdf/warehouse_robot.urdf.xacro (robot description, xacro)
@@ -5,5 +5,5 @@
   <!-- Chassis -->
   <xacro:property name="base_length" value="0.75"/>
-  <xacro:property name="base_width" value="0.75"/>
+  <xacro:property name="base_width" value="0.65"/>
   <xacro:property name="base_height" value="0.25"/>
   <xacro:property name="base_mass" value="16.0"/>
