Commit message: feat: bottom camera for floor tag detection

File: warehouse_sim/urdf/warehouse_robot.urdf.xacro (robot description, xacro)
@@ -9,9 +9,9 @@
   <xacro:property name="base_mass" value="16.0"/>
   <!-- Drive wheels -->
-  <xacro:property name="wheel_radius" value="0.1"/>
+  <xacro:property name="wheel_radius" value="0.13"/>
   <xacro:property name="wheel_width" value="0.06"/>
   <xacro:property name="wheel_mass" value="0.75"/>
   <!-- Caster wheels -->
-  <xacro:property name="caster_radius" value="0.05"/>
+  <xacro:property name="caster_radius" value="0.065"/>
   <xacro:property name="caster_mass" value="0.2"/>
   <!-- Cargo cage: thin walls around the chassis, front wall has a hinged flap -->
@@ -24,4 +24,7 @@
   <xacro:property name="camera_size" value="0.04"/>
   <xacro:property name="camera_mass" value="0.05"/>
+  <!-- Bottom-facing camera, for reading floor AprilTags -->
+  <xacro:property name="bottom_camera_size" value="0.03"/>
+  <xacro:property name="bottom_camera_mass" value="0.03"/>
   <!-- Front 2D lidar -->
   <xacro:property name="lidar_radius" value="0.05"/>
@@ -339,4 +342,59 @@
     </sensor>
   </gazebo>
+  <!-- Bottom camera: flush on the chassis underside, centered, pointing straight down
+       through the ground clearance gap to read floor AprilTags -->
+  <link name="bottom_camera_link">
+    <visual>
+      <geometry>
+        <box size="${bottom_camera_size} ${bottom_camera_size} ${bottom_camera_size}"/>
+      </geometry>
+      <material name="wheel_black"/>
+    </visual>
+    <collision>
+      <geometry>
+        <box size="${bottom_camera_size} ${bottom_camera_size} ${bottom_camera_size}"/>
+      </geometry>
+    </collision>
+    <inertial>
+      <mass value="${bottom_camera_mass}"/>
+      <inertia
+        ixx="${bottom_camera_mass / 6.0 * bottom_camera_size*bottom_camera_size}" ixy="0" ixz="0"
+        iyy="${bottom_camera_mass / 6.0 * bottom_camera_size*bottom_camera_size}" iyz="0"
+        izz="${bottom_camera_mass / 6.0 * bottom_camera_size*bottom_camera_size}"/>
+    </inertial>
+  </link>
+  <joint name="bottom_camera_joint" type="fixed">
+    <parent link="base_link"/>
+    <child link="bottom_camera_link"/>
+    <origin xyz="0 0 ${-(base_height/2 + bottom_camera_size/2)}" rpy="0 ${pi/2} 0"/>
+  </joint>
+  <link name="bottom_camera_optical_frame"/>
+  <joint name="bottom_camera_optical_joint" type="fixed">
+    <parent link="bottom_camera_link"/>
+    <child link="bottom_camera_optical_frame"/>
+    <origin xyz="0 0 0" rpy="${-pi/2} 0 ${-pi/2}"/>
+  </joint>
+  <gazebo reference="bottom_camera_link">
+    <material>Gazebo/Black</material>
+    <sensor name="bottom_camera" type="camera">
+      <camera>
+        <horizontal_fov>1.9</horizontal_fov>
+        <image>
+          <width>640</width>
+          <height>480</height>
+        </image>
+        <clip>
+          <!-- Lens sits only a couple cm off the floor, so the near plane has to be tiny -->
+          <near>0.005</near>
+          <far>1.0</far>
+        </clip>
+        <optical_frame_id>bottom_camera_optical_frame</optical_frame_id>
+      </camera>
+      <always_on>true</always_on>
+      <update_rate>15</update_rate>
+      <visualize>true</visualize>
+      <topic>bottom_camera</topic>
+    </sensor>
+  </gazebo>
   <!-- IMU: mounted at the chassis origin -->
   <link name="imu_link">

Commit message: fix: pull back bottom camera for better tag visibility

File: warehouse_sim/urdf/warehouse_robot.urdf.xacro (robot description, xacro)
@@ -27,4 +27,7 @@
   <xacro:property name="bottom_camera_size" value="0.03"/>
   <xacro:property name="bottom_camera_mass" value="0.03"/>
+  <!-- Height of the lens above the floor: bigger gap widens the footprint the camera
+       sees on the ground, so a tag stays in frame longer as the robot drives over it -->
+  <xacro:property name="bottom_camera_ground_gap" value="0.03"/>
   <!-- Front 2D lidar -->
   <xacro:property name="lidar_radius" value="0.05"/>
@@ -40,4 +43,5 @@
   <xacro:property name="caster_z_offset" value="${caster_radius - base_z}"/>
   <xacro:property name="caster_x_offset" value="${base_length / 2 - caster_radius - 0.02}"/>
+  <xacro:property name="bottom_camera_z_offset" value="${bottom_camera_ground_gap + bottom_camera_size/2 - base_z}"/>
   <xacro:property name="cage_base_z" value="${base_height / 2.0}"/>
   <xacro:property name="cage_front_upper_height" value="${cage_wall_height - cage_flap_height}"/>
@@ -367,5 +371,5 @@
     <parent link="base_link"/>
     <child link="bottom_camera_link"/>
-    <origin xyz="0 0 ${-(base_height/2 + bottom_camera_size/2)}" rpy="0 ${pi/2} 0"/>
+    <origin xyz="0 0 ${bottom_camera_z_offset}" rpy="0 ${pi/2} 0"/>
   </joint>
   <link name="bottom_camera_optical_frame"/>

Commit message: feat: various EKF improvements

File: warehouse_sim/urdf/warehouse_robot.urdf.xacro (robot description, xacro)
@@ -29,5 +29,5 @@
   <!-- Height of the lens above the floor: bigger gap widens the footprint the camera
        sees on the ground, so a tag stays in frame longer as the robot drives over it -->
-  <xacro:property name="bottom_camera_ground_gap" value="0.03"/>
+  <xacro:property name="bottom_camera_ground_gap" value="0.043"/>
   <!-- Front 2D lidar -->
   <xacro:property name="lidar_radius" value="0.05"/>
@@ -396,5 +396,5 @@
       </camera>
       <always_on>true</always_on>
-      <update_rate>15</update_rate>
+      <update_rate>30</update_rate>
       <visualize>true</visualize>
       <topic>bottom_camera</topic>

Commit message: feat: internal conveyer belt

File: warehouse_sim/urdf/warehouse_robot.urdf.xacro (robot description, xacro)
@@ -21,4 +21,7 @@
   <xacro:property name="cage_wall_mass" value="0.5"/>
   <xacro:property name="cage_flap_mass" value="0.3"/>
+  <!-- Cage floor: doubles as an ejector belt (gz-sim TrackController) -->
+  <xacro:property name="cage_floor_thickness" value="0.01"/>
+  <xacro:property name="cage_floor_mass" value="0.4"/>
   <!-- Rear RGB camera -->
   <xacro:property name="camera_size" value="0.04"/>
@@ -46,4 +49,6 @@
   <xacro:property name="cage_base_z" value="${base_height / 2.0}"/>
   <xacro:property name="cage_front_upper_height" value="${cage_wall_height - cage_flap_height}"/>
+  <xacro:property name="cage_floor_length" value="${base_length - 2*cage_wall_thickness}"/>
+  <xacro:property name="cage_floor_width" value="${base_width - 2*cage_wall_thickness}"/>
   <material name="body_gray">
     <color rgba="0.3 0.3 0.3 1.0"/>
@@ -240,4 +245,45 @@
     <material>Gazebo/Black</material>
   </gazebo>
+  <!-- Cage floor: sits on the chassis roof inside the cage walls. It's also the ejector
+       belt surface — TrackController drives its contact velocity to push cargo resting
+       on it out through the (opened) front flap. -->
+  <link name="cage_floor_link">
+    <visual>
+      <geometry>
+        <box size="${cage_floor_length} ${cage_floor_width} ${cage_floor_thickness}"/>
+      </geometry>
+      <material name="wheel_black"/>
+    </visual>
+    <collision>
+      <geometry>
+        <box size="${cage_floor_length} ${cage_floor_width} ${cage_floor_thickness}"/>
+      </geometry>
+    </collision>
+    <inertial>
+      <mass value="${cage_floor_mass}"/>
+      <inertia
+        ixx="${cage_floor_mass / 12.0 * (cage_floor_width*cage_floor_width + cage_floor_thickness*cage_floor_thickness)}" ixy="0" ixz="0"
+        iyy="${cage_floor_mass / 12.0 * (cage_floor_length*cage_floor_length + cage_floor_thickness*cage_floor_thickness)}" iyz="0"
+        izz="${cage_floor_mass / 12.0 * (cage_floor_length*cage_floor_length + cage_floor_width*cage_floor_width)}"/>
+    </inertial>
+  </link>
+  <joint name="cage_floor_joint" type="fixed">
+    <parent link="base_link"/>
+    <child link="cage_floor_link"/>
+    <origin xyz="0 0 ${cage_base_z + cage_floor_thickness/2}" rpy="0 0 0"/>
+  </joint>
+  <!-- Fixed joints get lumped into their parent by the URDF->SDF conversion, which would
+       merge cage_floor_link into base_link and leave TrackController nothing to reference -->
+  <gazebo reference="cage_floor_joint">
+    <disableFixedJointLumping>true</disableFixedJointLumping>
+  </gazebo>
+  <gazebo reference="cage_floor_link">
+    <material>Gazebo/DarkGrey</material>
+    <mu1>1.0</mu1>
+    <mu2>1.0</mu2>
+    <!-- Perpendicular to the belt's travel direction (link +x, toward the flap), so
+         TrackController has a well-defined friction axis to apply drive velocity along -->
+    <fdir1>0 1 0</fdir1>
+  </gazebo>
   <!-- Front lidar: centered on the chassis front face, below the cage, so half the puck
        sticks out past the front edge -->
@@ -460,4 +506,13 @@
     </plugin>
   </gazebo>
+  <!-- Ejector belt: velocity-only, commanded over gz transport (not ros2_control) on
+       /model/warehouse_robot/link/cage_floor_link/track_cmd_vel, bridged to ROS in
+       sim.launch.py. Positive velocity pushes cargo out the front (+x, flap side). -->
+  <gazebo>
+    <plugin filename="gz-sim-track-controller-system" name="gz::sim::systems::TrackController">
+      <link>cage_floor_link</link>
+      <odometry_publish_frequency>10</odometry_publish_frequency>
+    </plugin>
+  </gazebo>
   <!-- Ground-truth pose for testing: publishes only the robot model's pose (no links/
        sensors/collisions) to /model/warehouse_robot/pose, bridged to ROS in sim.launch.py -->

Commit message: chore: remove rear camera

File: warehouse_sim/urdf/warehouse_robot.urdf.xacro (robot description, xacro)
@@ -24,7 +24,4 @@
   <xacro:property name="cage_floor_thickness" value="0.01"/>
   <xacro:property name="cage_floor_mass" value="0.4"/>
-  <!-- Rear RGB camera -->
-  <xacro:property name="camera_size" value="0.04"/>
-  <xacro:property name="camera_mass" value="0.05"/>
   <!-- Bottom-facing camera, for reading floor AprilTags -->
   <xacro:property name="bottom_camera_size" value="0.03"/>
@@ -337,59 +334,4 @@
     </sensor>
   </gazebo>
-  <!-- Rear camera: mounted flush on the chassis back face, pointing straight out along -x -->
-  <link name="rear_camera_link">
-    <visual>
-      <geometry>
-        <box size="${camera_size} ${camera_size} ${camera_size}"/>
-      </geometry>
-      <material name="wheel_black"/>
-    </visual>
-    <collision>
-      <geometry>
-        <box size="${camera_size} ${camera_size} ${camera_size}"/>
-      </geometry>
-    </collision>
-    <inertial>
-      <mass value="${camera_mass}"/>
-      <inertia
-        ixx="${camera_mass / 6.0 * camera_size*camera_size}" ixy="0" ixz="0"
-        iyy="${camera_mass / 6.0 * camera_size*camera_size}" iyz="0"
-        izz="${camera_mass / 6.0 * camera_size*camera_size}"/>
-    </inertial>
-  </link>
-  <joint name="rear_camera_joint" type="fixed">
-    <parent link="base_link"/>
-    <child link="rear_camera_link"/>
-    <origin xyz="${-(base_length/2 + camera_size/2)} 0 0" rpy="0 0 ${pi}"/>
-  </joint>
-  <!-- Optical frame: REP 103 convention (Z forward, X right, Y down), used for image/camera_info -->
-  <link name="rear_camera_optical_frame"/>
-  <joint name="rear_camera_optical_joint" type="fixed">
-    <parent link="rear_camera_link"/>
-    <child link="rear_camera_optical_frame"/>
-    <origin xyz="0 0 0" rpy="${-pi/2} 0 ${-pi/2}"/>
-  </joint>
-  <gazebo reference="rear_camera_link">
-    <material>Gazebo/Black</material>
-    <sensor name="rear_camera" type="camera">
-      <camera>
-        <horizontal_fov>1.4</horizontal_fov>
-        <image>
-          <width>640</width>
-          <height>480</height>
-        </image>
-        <clip>
-          <near>0.05</near>
-          <far>50</far>
-        </clip>
-        <!-- Sensor is aimed straight out the back for now; revisit if the mount angle changes -->
-        <optical_frame_id>rear_camera_optical_frame</optical_frame_id>
-      </camera>
-      <always_on>true</always_on>
-      <update_rate>15</update_rate>
-      <visualize>true</visualize>
-      <topic>rear_camera</topic>
-    </sensor>
-  </gazebo>
   <!-- Bottom camera: flush on the chassis underside, centered, pointing straight down
        through the ground clearance gap to read floor AprilTags -->
